File: esp32-smartwatch.kicad_pcb (KiCad board)
At the start: 4 copper layers, 37.5 x 37.5 mm, 54 parts, among them J1 USB_B_Micro, J2 LiPo_JST, M1 316040001, Q1 SI1317DL-T1-GE3, Q2 BSS123, Q3 BSS123, U1 BMA400, U2 TPD3E001DRLR, U3 XC6220B331MR, U4 CH340E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

Commit message: updated images
Connections:
- U3 pad 3: Net-(U3-Pad3) -> Net-(C4-Pad1)
Routing:
- net Net-(C4-Pad1): track 6.64 -> 10.5 mm
- net /~TFT_CS: track 29.0 -> 30.6 mm
- net /SDA: track 32.9 -> 31.7 mm
- net GND: track 63.7 -> 64.6 mm, vias 52 -> 47
- net +3V3: track 35.3 -> 35.9 mm
- net /BTN1: vias 3 -> 2
Other:
- net class Default: via_dia 0.4 -> 0.5; via_drill 0.2 -> 0.25
- net class i2c: via_dia 0.4 -> 0.5; via_drill 0.2 -> 0.25
- rule via_min_drill: 0.2 -> 0.25
- rule via_min_size: 0.4 -> 0.5
- board text added: "JLCJLCJLCJLC"
- board text added: "Smartwatch Timothy Nguyen Rev B"
- board text removed: "Smartwatch Rev 1.1"
