File: esp32-smartwatch.kicad_pcb (KiCad board)
At the start: 4 copper layers, 37.5 x 37.5 mm, 54 parts, among them J1 USB_B_Micro, J2 LiPo_JST, M1 316040001, Q1 SI1317DL-T1-GE3, Q2 BSS123, Q3 BSS123, U1 BMA400, U2 TPD3E001DRLR, U3 XC6220B331MR, U4 CH340E, U5 DS3231MZ, U6 TPS3831, U7 MCP73831-2-OT, U8 ttgo-32-micro, U9 GC9A01_IPS_display_SPI

Commit message: Redoing PCB
Parts:
- removed 3V3: +3V3, TestPoint:TestPoint_THTPad_D1.0mm_Drill0.5mm
- removed BOOT: BOOT, custom-footprints:switch
- removed C16, C17: 0.1uF, Capacitor_SMD:C_0603_1608Metric
- removed GND: GND, TestPoint:TestPoint_THTPad_D1.0mm_Drill0.5mm
- removed LED: STATUS, LED_SMD:LED_0603_1608Metric
- removed M1: 316040001, custom-footprints:Custom-pad
- removed R6: 100K, Resistor_SMD:R_0603_1608Metric
- removed RST: ~RST, custom-footprints:switch
- removed U9: GC9A01_IPS_display_SPI, open-Smartwatch:GC9A01_IPS_display_under
- removed VBAT: VBAT, TestPoint:TestPoint_THTPad_D1.0mm_Drill0.5mm
- removed VBUS: VBUS, TestPoint:TestPoint_THTPad_D1.0mm_Drill0.5mm
- added BOOT1: SW1, custom-footprints:switch, F.Cu at (157.2, 100.6)
- added D2: STATUS, LED_SMD:LED_0603_1608Metric, F.Cu at (179.4, 81.4)
- added LS1: ‎SMT-0340-T-R‎, custom-footprints:SMT-0340-T-R, F.Cu at (183.6, 93.6)
- added R12: 150, Resistor_SMD:R_0603_1608Metric, F.Cu at (179.4, 90.5)
- added R15: 22, Resistor_SMD:R_0603_1608Metric, F.Cu at (165.0, 92.6)
- added R16: 10K, Resistor_SMD:R_0603_1608Metric, F.Cu at (179.4, 96.3)
- added RST1: SW2, custom-footprints:switch, F.Cu at (156.5, 78.0)
- added TP1: VBUS, TestPoint:TestPoint_THTPad_D1.0mm_Drill0.5mm, F.Cu at (152.2, 83.8)
- added TP2: VBAT, TestPoint:TestPoint_THTPad_D1.0mm_Drill0.5mm, F.Cu at (161.1, 103.7)
- added TP3: +3V3, TestPoint:TestPoint_THTPad_D1.0mm_Drill0.5mm, F.Cu at (184.5, 96.8)
- added TP4: GND, TestPoint:TestPoint_THTPad_D1.0mm_Drill0.5mm, F.Cu at (176.6, 104.2)
- BTN1: value BTN1 -> SW3
- BTN2: value BTN2 -> SW4
- C1, C10, C12, C2, C6: footprint Capacitor_SMD:C_0603_1608Metric -> Capacitor_SMD:C_0402_1005Metric
- C11, C5: value 0.1uF -> 4.7uF; footprint Capacitor_SMD:C_0603_1608Metric -> Capacitor_SMD:C_0402_1005Metric
- C13: value 4.7uF -> 0.1uF; footprint Capacitor_SMD:C_0603_1608Metric -> Capacitor_SMD:C_0402_1005Metric
- C3, C8: value 0.1uF -> 10uF
- C4, C7, C9: value 10uF -> 0.1uF; footprint Capacitor_SMD:C_0805_2012Metric -> Capacitor_SMD:C_0402_1005Metric
- D1, D3: value MBR0520 -> MBR120LSF
- J2: footprint custom-footprints:Custom-pad -> custom-footprints:Custom_pad
- R10: value 330 -> 150
- R11, R13: value 10K -> 330
- R14: value 100K -> 10K
- R4: value 4.7K -> 10K
- R5: value 100K -> 4.7K
- R7: value 2K -> 100K
- R8: value 150 -> 100K
- R9: value 150 -> 330
- U1: value BMA400 -> BMA423; footprint open-Smartwatch:LGA-12_2x2mm_P0.5mm -> custom-footprints:IC_BMA400
- U6: value TPS3831 -> MCP73831-2-OT; footprint Package_SON:Texas_X2SON-4_1x1mm_P0.65mm -> Package_TO_SOT_SMD:SOT-23-5
- U7: value MCP73831-2-OT -> ttgo-32-micro; footprint Package_TO_SOT_SMD:SOT-23-5 -> open-Smartwatch:ttgo-32-micro
- U8: value ttgo-32-micro -> GC9A01_IPS_display_SPI; footprint open-Smartwatch:ttgo-32-micro -> open-Smartwatch:GC9A01_IPS_display_under; moved to B.Cu
- moved R14 33.3 mm to (186.2, 85.3), turned to 90 degrees
- moved C8 33.0 mm to (159.6, 74.4), turned to 90 degrees
- moved C4 26.8 mm to (185.8, 87.8), turned to 270 degrees
- moved D3 24.9 mm to (183.3, 90.5)
- moved Q3 23.4 mm to (179.6, 93.5)
- moved R13 23.4 mm to (159.2, 81.7), turned to 0 degrees
- moved U7 22.9 mm to (168.9, 79.3), turned to 0 degrees
- moved J1 22.2 mm to (153.5, 89.0), turned to 270 degrees
- moved U8 22.1 mm to (169.3, 101.5)
- moved R11 22.0 mm to (164.9, 99.1), turned to 0 degrees
- moved C11 21.9 mm to (171.5, 98.3), turned to 0 degrees
- moved U6 21.7 mm to (172.3, 95.8)
- moved R3 21.0 mm to (159.2, 84.7), turned to 0 degrees
- moved C2 20.2 mm to (157.4, 87.2), turned to 180 degrees
- moved R9 19.6 mm to (179.4, 83.0)
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Connections:
- net /M- renamed Net-(D3-Pad2)
- C1 pad 1: VBUS -> GND
- C1 pad 2: GND -> +3V3
- C10 pad 1: +3V3 -> /~RST
- C11 pad 1: +3V3 -> VBUS
- C12 pad 1: VBUS -> VBAT
- C13 pad 1: VBAT -> +3V3
- C2 pad 1: GND -> VBUS
- C2 pad 2: +3V3 -> GND
- C3 pad 1: GND -> Net-(C3-Pad1)
- C3 pad 2: VBUS -> GND
- C4 pad 1: Net-(C4-Pad1) -> +3V3
- C5 pad 1: GND -> +3V3
- C5 pad 2: Net-(C5-Pad2) -> GND
- C6 pad 1: +3V3 -> GND
- C6 pad 2: GND -> +3V3
- D1 pad 1: Net-(C4-Pad1) -> Net-(C3-Pad1)
- D3 pad 1: /M+ -> +3V3
- Q1 pad 2: Net-(C4-Pad1) -> Net-(C3-Pad1)
- R10 pad 1: +3V3 -> /LEDK
- R10 pad 2: /M+ -> Net-(Q2-Pad1)
- R11 pad 1: +3V3 -> Net-(BOOT1-Pad2)
- R11 pad 2: /BTN1 -> /BOOT
- R13 pad 1: +3V3 -> Net-(R13-Pad1)
- R13 pad 2: /BTN2 -> /~RST
- R14 pad 2: /BAT_STAT -> /BTN1
- R4 pad 1: Net-(R4-Pad1) -> +3V3
- R4 pad 2: GND -> /~RST
- R5 pad 1: VBAT -> Net-(R5-Pad1)
- R5 pad 2: /BAT_LVL -> GND
- R7 pad 1: Net-(D2-Pad1) -> VBAT
- R7 pad 2: GND -> /BAT_LVL
- R8 pad 1: /LEDK -> /BAT_LVL
- R8 pad 2: Net-(Q2-Pad1) -> GND
- R9 pad 1: /PWM -> Net-(D2-Pad1)
- R9 pad 2: Net-(Q3-Pad1) -> GND
- U3 pad 1: Net-(C4-Pad1) -> Net-(C3-Pad1)
- U3 pad 3: Net-(C4-Pad1) -> Net-(C3-Pad1)
- U4 pad 10: Net-(C5-Pad2) -> +3V3
- U4 pad 7: VBUS -> +3V3
- U4 pad 8: /TXD0 -> /RXD0
- U4 pad 9: /RXD0 -> /TXD0
- U5 pad 4: Net-(U5-Pad4) -> /~DS_RST
- U6 pad 1: /~RST -> /BAT_STAT
- U6 pad 2: /~MR -> GND
- U6 pad 3: GND -> VBAT
- U6 pad 4: +3V3 -> VBUS
- U6 pad 5: GND -> Net-(R5-Pad1)
- U7 pad 1: /BAT_STAT -> GND
- U7 pad 2: GND -> +3V3
- U7 pad 3: VBAT -> /~RST
- U7 pad 4: VBUS -> Net-(U7-Pad4)
- U7 pad 5: Net-(R4-Pad1) -> Net-(U7-Pad5)
- U8 pad 10: /~TFT_RST -> /MOSI
- U8 pad 11: /BTN1 -> /~TFT_RST
- U8 pad 12: /BTN2 -> GND
- U8 pad 2: +3V3 -> Net-(Q2-Pad3)
- U8 pad 3: /~RST -> Net-(R15-Pad2)
- U8 pad 4: Net-(U8-Pad4) -> +3V3
- U8 pad 5: Net-(U8-Pad5) -> GND
- U8 pad 6: /BAT_LVL -> GND
- U8 pad 7: /BAT_STAT -> /TFT_DC
- U8 pad 8: /LEDK -> /~TFT_CS
- U8 pad 9: /PWM -> /SCLK
Routing:
- net GND: track 64.6 -> 0.00 mm, vias 47 -> 0
- net VBUS: track 46.4 -> 0.00 mm, vias 2 -> 0
- net /~TFT_RST: track 37.5 -> 0.00 mm, vias 1 -> 0
- net +3V3: track 35.9 -> 0.00 mm, vias 25 -> 0
- net /BOOT: track 35.5 -> 0.00 mm, vias 3 -> 0
- net /BTN1: track 35.0 -> 0.00 mm, vias 2 -> 0
- net /BAT_STAT: track 33.2 -> 0.00 mm, vias 2 -> 0
- net /SDA: track 31.7 -> 0.00 mm, vias 2 -> 0
- net /~TFT_CS: track 30.6 -> 0.00 mm, vias 3 -> 0
- net /~DS_INT: track 29.0 -> 0.00 mm, vias 2 -> 0
- net /SCLK: track 28.9 -> 0.00 mm, vias 1 -> 0
- net /MOSI: track 28.8 -> 0.00 mm, vias 1 -> 0
- net /BAT_LVL: track 28.7 -> 0.00 mm, vias 2 -> 0
- net /BTN2: track 27.4 -> 0.00 mm, vias 2 -> 0
- net /TXD0: track 27.0 -> 0.00 mm, vias 2 -> 0
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- removed copper zone on F.Cu, net +3V3
- removed copper zone on In2.Cu, net +3V3
- removed copper zone on F.Cu, net GND
- removed copper zone on In1.Cu, net GND
Other:
- board text removed: "+"
- board text removed: "JLCJLCJLCJLC"
- board text removed: "Smartwatch Timothy Nguyen Rev B"

Commit message: PCB layout Rev C
Parts:
- removed D2: STATUS, LED_SMD:LED_0603_1608Metric
- removed RST1: SW2, custom-footprints:switch
- removed TP2: VBAT, TestPoint:TestPoint_THTPad_D1.0mm_Drill0.5mm
- added LED: STATUS, LED_SMD:LED_0603_1608Metric, F.Cu at (179.4, 81.4)
- added RST: SW2, custom-footprints:switch, F.Cu at (156.3, 78.1)
- added VBAT: VBAT, TestPoint:TestPoint_THTPad_D1.0mm_Drill0.5mm, F.Cu at (161.8, 104.5)
- C13: moved to B.Cu
- moved 3V3 34.0 mm to (153.3, 83.2)
- moved VBUS 12.4 mm to (153.7, 96.1)
- moved R13 1.41 mm to (158.1, 82.5)
- moved R3 1.41 mm to (158.1, 85.5)
- moved R4 1.41 mm to (158.1, 84.0)
- moved D1 1.05 mm to (157.2, 94.7)
- moved C10 0.99 mm to (158.7, 81.2)
- moved R11 0.76 mm to (164.4, 98.6)
- moved C9 0.66 mm to (160.9, 73.2)
- moved C13 0.34 mm to (168.1, 99.4)
- moved Q1 0.09 mm to (159.6, 96.3)
- moved C5 0.07 mm to (166.4, 96.8)
- moved C8 0.06 mm to (159.6, 74.4)
- renumbered TP3 to 3V3, BOOT1 to BOOT, TP4 to GND, TP1 to VBUS
Connections:
- BTN1 pad 4: (no net) -> /BTN1
- U7 pad EP: (no net) -> GND
Routing:
- net GND: track 0.00 -> 58.5 mm, vias 0 -> 53
- net VBAT: track 0.00 -> 50.4 mm, vias 0 -> 8
- net VBUS: track 0.00 -> 48.5 mm, vias 0 -> 1
- net +3V3: track 0.00 -> 42.6 mm, vias 0 -> 18
- net /BTN1: track 0.00 -> 36.9 mm, vias 0 -> 3
- net /SCLK: track 0.00 -> 33.1 mm, vias 0 -> 1
- net /MOSI: track 0.00 -> 33.0 mm, vias 0 -> 1
- net /TXD0: track 0.00 -> 28.4 mm, vias 0 -> 2
- net /~TFT_RST: track 0.00 -> 28.3 mm, vias 0 -> 2
- net /RXD0: track 0.00 -> 27.7 mm, vias 0 -> 2
- net /BAT_LVL: track 0.00 -> 27.6 mm, vias 0 -> 2
- net /BOOT: track 0.00 -> 26.7 mm, vias 0 -> 2
- net /SCL: track 0.00 -> 26.4 mm, vias 0 -> 4
- net /BTN2: track 0.00 -> 24.6 mm, vias 0 -> 2
- net /~TFT_CS: track 0.00 -> 24.1 mm, vias 0 -> 1
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- added copper zone on In2.Cu, net +3V3
- added copper zone on In1.Cu, net GND
Other:
- board text added: "+"
- board text added: "ESP32 Smartwatch Timothy Nguyen Rev. C"
- board text added: "JLCJLCJLCJLC"
