File: esp32-smartwatch.sch (KiCad schematic (older format))
At the start: 54 parts, among them J1 USB_B_Micro, J2 LiPo_JST, M1 316040001, Q1 SI1317DL-T1-GE3, Q2 BSS123, Q3 BSS123, U1 BMA400, U2 TPD3E001DRLR, U3 XC6220B331MR, U4 CH340E, U5 DS3231MZ, U6 TPS3831, U7 MCP73831-2-OT, U8 ttgo-32-micro, U9 GC9A01_IPS_display_SPI

Commit message: updated images
Connections:
- net at C4.1, D1.1 (K), Q1.2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: now also U3.3 (CE)
- no-connect marks 21 -> 20
Other:
- moved on the sheet: C4
Changed lines of the file:
@@
 Title "Personal ESP32 Smartwatch"
 Date "2021-06-18"
-Rev "1.0"
+Rev "B"
 Comp ""
 Comment1 ""
@@
 Wire Notes Line
 	4450 500  4450 7800
-Wire Wire Line
-	2000 6950 2150 6950
-Connection ~ 2000 6950
-Wire Wire Line
-	2000 7000 2000 6950
+Connection ~ 1950 6950
+Wire Wire Line
+	1950 7000 1950 6950
 Connection ~ 1800 6950
 Wire Wire Line
-	1800 6950 2000 6950
-Wire Wire Line
-	2000 7300 2000 7350
+	1800 6950 1950 6950
+Wire Wire Line
+	1950 7300 1950 7350
 $Comp
 L Device:C C4
 U 1 1 6143BFCB
-P 2000 7150
-F 0 "C4" H 1750 7150 50  0000 L CNN
-F 1 "10uF" H 1700 7050 50  0000 L CNN
-F 2 "Capacitor_SMD:C_0805_2012Metric" H 2038 7000 50  0001 C CNN
-F 3 "~" H 2000 7150 50  0001 C CNN
-	1    2000 7150
+P 1950 7150
+F 0 "C4" H 1700 7150 50  0000 L CNN
+F 1 "10uF" H 1650 7050 50  0000 L CNN
+F 2 "Capacitor_SMD:C_0805_2012Metric" H 1988 7000 50  0001 C CNN
+F 3 "~" H 1950 7150 50  0001 C CNN
+	1    1950 7150
 	1    0    0    -1
 $EndComp
@@
 L power:GND #PWR014
 U 1 1 614608F8
-P 2000 7350
-F 0 "#PWR014" H 2000 7100 50  0001 C CNN
-F 1 "GND" H 2005 7177 50  0001 C CNN
-F 2 "" H 2000 7350 50  0001 C CNN
-F 3 "" H 2000 7350 50  0001 C CNN
-	1    2000 7350
+P 1950 7350
+F 0 "#PWR014" H 1950 7100 50  0001 C CNN
+F 1 "GND" H 1955 7177 50  0001 C CNN
+F 2 "" H 1950 7350 50  0001 C CNN
+F 3 "" H 1950 7350 50  0001 C CNN
+	1    1950 7350
 	1    0    0    -1
 $EndComp
@@
 	3500 6700 3500 6950
 $Comp
-L Regulator_Linear:XC6220B331MR U3
-U 1 1 60D93332
-P 2650 7050
-F 0 "U3" H 2650 7417 50  0000 C CNN
-F 1 "XC6220B331MR" H 2650 7326 50  0000 C CNN
-F 2 "Package_TO_SOT_SMD:SOT-23-5" H 2650 7050 50  0001 C CNN
-F 3 "https://www.torexsemi.com/file/xc6220/XC6220.pdf" H 3400 6050 50  0001 C CNN
-	1    2650 7050
-	1    0    0    -1
-$EndComp
-$Comp
 L Device:C C7
 U 1 1 60D9AEE4
@@
 Wire Wire Line
 	3150 6950 3200 6950
-NoConn ~ 2150 7150
 $Comp
 L power:VBUS #PWR04
@@
 	1    0    0    -1
 $EndComp
+$Comp
+L Regulator_Linear:XC6220B331MR U3
+U 1 1 60D93332
+P 2650 7050
+F 0 "U3" H 2650 7417 50  0000 C CNN
+F 1 "XC6220B331MR" H 2650 7326 50  0000 C CNN
+F 2 "Package_TO_SOT_SMD:SOT-23-5" H 2650 7050 50  0001 C CNN
+F 3 "https://www.torexsemi.com/file/xc6220/XC6220.pdf" H 3400 6050 50  0001 C CNN
+	1    2650 7050
+	1    0    0    -1
+$EndComp
+Wire Wire Line
+	1950 6950 2100 6950
+Wire Wire Line
+	2150 7150 2100 7150
+Wire Wire Line
+	2100 7150 2100 6950
+Connection ~ 2100 6950
+Wire Wire Line
+	2100 6950 2150 6950
 $EndSCHEMATC

Commit message: Redoing PCB
Parts:
- removed C11, C16, C17, C5: 0.1uF, Capacitor_SMD:C_0603_1608Metric, symbol Device:C
- removed M1: 316040001, custom-footprints:Custom-pad, symbol Motor:Motor_DC_ALT
- removed R10: 330, Resistor_SMD:R_0603_1608Metric, symbol Device:R
- removed R14: 100K, Resistor_SMD:R_0603_1608Metric, symbol Device:R
- removed R9: 150, Resistor_SMD:R_0603_1608Metric, symbol Device:R
- removed U6: TPS3831, Package_SON:Texas_X2SON-4_1x1mm_P0.65mm, symbol Power_Supervisor:TPS3831
- added C10, C13: 0.1uF, Capacitor_SMD:C_0402_1005Metric, symbol Device:C
- added LS1: ‎SMT-0340-T-R‎, custom-footprints:SMT-0340-T-R, symbol Device:Speaker
- added R11, R13: 330, Resistor_SMD:R_0603_1608Metric, symbol Device:R
- added R12: 150, Resistor_SMD:R_0603_1608Metric, symbol Device:R
- added R15: 22, Resistor_SMD:R_0603_1608Metric, symbol Device:R
- added R4: 10K, Resistor_SMD:R_0603_1608Metric, symbol Device:R
- C1: renamed from C2; footprint Capacitor_SMD:C_0603_1608Metric -> Capacitor_SMD:C_0402_1005Metric
- C11: renamed from C12; footprint Capacitor_SMD:C_0603_1608Metric -> Capacitor_SMD:C_0402_1005Metric
- C12: renamed from C13; footprint Capacitor_SMD:C_0603_1608Metric -> Capacitor_SMD:C_0402_1005Metric
- C2: renamed from C1; footprint Capacitor_SMD:C_0603_1608Metric -> Capacitor_SMD:C_0402_1005Metric
- C3: renamed from C4; footprint Capacitor_SMD:C_0805_2012Metric -> Capacitor_SMD:C_0603_1608Metric
- C4: renamed from C6; footprint Capacitor_SMD:C_0603_1608Metric -> Capacitor_SMD:C_0402_1005Metric
- C5: renamed from C7; value 10uF -> 4.7uF; footprint Capacitor_SMD:C_0805_2012Metric -> Capacitor_SMD:C_0402_1005Metric
- C6: renamed from C3; footprint Capacitor_SMD:C_0603_1608Metric -> Capacitor_SMD:C_0402_1005Metric
- C7: renamed from C8; footprint Capacitor_SMD:C_0603_1608Metric -> Capacitor_SMD:C_0402_1005Metric
- C8: renamed from C9; footprint Capacitor_SMD:C_0805_2012Metric -> Capacitor_SMD:C_0603_1608Metric
- C9: renamed from C10; footprint Capacitor_SMD:C_0603_1608Metric -> Capacitor_SMD:C_0402_1005Metric
- D1, D3: value MBR0520 -> MBR120LSF
- J2: footprint custom-footprints:Custom-pad -> custom-footprints:Custom_pad
- R9: renamed from R7; value 2K -> 330
- U1: value BMA400 -> BMA423; footprint open-Smartwatch:LGA-12_2x2mm_P0.5mm -> custom-footprints:IC_BMA400
- renumbered BOOT to BOOT1, R8 to R10, R11 to R14, R13 to R16, R4 to R5, R5 to R7, R6 to R8, RST to RST1, U7 to U6, U8 to U7, U9 to U8
Connections:
- net M+ is gone; now on net +3V3: D3.1 (K)
- net +3V3: now also C6.2, U4.10 (V3), U4.7 (VCC), C13.1, LS1.1, R15.1, R4.1; no longer U8.3 (LEDA)
- net BAT_STAT: now also U7.27 (IO16); no longer U7.7 (IO35)
- net BOOT: now also R11.2; no longer BOOT1.2
- net BTN1: now also U7.16 (IO13); no longer U7.11 (IO26)
- net BTN2: now also U7.23 (MTDO); no longer U7.12 (IO27)
- net GND: now also C10.2, C13.2
- net RXD0: now also U4.8 (TXD); no longer U4.9 (RXD)
- net TXD0: now also U4.9 (RXD); no longer U4.8 (TXD)
- net VBUS: no longer C6.2, U4.7 (VCC)
- net ~RST: now also C10.1, R13.2, R4.2
- net ~DS_RST: now reaches U7.28 (IO17)
- net ~DS_RST: now also U5.4 (~RST)
- net IO19: now reaches D2.2 (A), U7.31 (IO19)
- net at Q3.1 (G): now also R12.2
- net M-: no longer names the net of D3.2 (A), Q3.3 (D)
- net M-: now also LS1.2
- net PWM renamed ALARM
- net ALARM: now also R12.1
- net ~MR: no longer names the net of RST1.2
- net ~MR: now also R13.1
- new net: BOOT1.2, R11.1
- new net: R15.2, U8.3 (LEDA)
- no-connect marks 20 -> 18
Other:
- note added: "50% PWM"
- note added: "Buzzer\n\n\n"
- note added: "CHIP_ID: \n0x68\n\n\n\n"
- note added: "CHIP_ID:\n0x13\n"
- note added: "Configure VSPI (SPI3) to\nbypass GPIO matrix."
- note added: "Enable internal \npull-up for \n~DS_INT and BAT_STAT."
- note added: "Internal SPI flash uses pins 17-22 (GPIO6-11). \nLeave disconnected."
- note added: "LEDK turns backlight on/off."
- note removed: "I2C_addr: \n0x14\n"
- note removed: "I2C_addr: \n0x68\n\n\n\n"
- note removed: "Manual reset input."
- note removed: "Vibration Motor"
- note removed: "Voltage Supervisor\n"
- note removed: "Vthres = 3.08 V"
- moved on the sheet: BOOT1, BTN1, BTN2, C8, C9, R14, R16, RST1

Commit message: Revised schematic
Other:
- note added: "Enable internal \npull-up for IO14 and IO16."
- note removed: "Enable internal \npull-up for \n~DS_INT and BAT_STAT."
Changed lines of the file:
@@
 Text Label 5300 4300 0    50   ~ 0
 ALARM
-Text Notes 6900 3100 0    50   ~ 0
+Text Notes 6800 3050 0    50   ~ 0
 Configure VSPI (SPI3) to\nbypass GPIO matrix.
 $Comp
@@
 	6950 4600 7300 4600
 NoConn ~ 5650 4100
-Text Notes 6900 2800 0    50   ~ 0
-Enable internal \npull-up for \n~DS_INT and BAT_STAT.
 Wire Wire Line
 	3100 2300 3400 2300
@@
 Text Label 7300 4500 2    50   ~ 0
 ~DS_RST
+Text Notes 6800 2750 0    50   ~ 0
+Enable internal \npull-up for IO14 and IO16.
 $EndSCHEMATC
